Commit message: modified:   src/mapping/mapping/grid_publisher.py 	modified:   src/odometry/odometry/odometry.py

File: src/snow_description/urdf/snow.urdf (robot description, URDF)
Before this commit: robot snow, 26 links, 25 joints
Links:
- removed link base_footprint_link
- added link mobile_base_link; visual box size=0.375 0.2667 0.07
- link base_link: geometry 
Joints:
- joint arm_base_joint: parent base_link -> mobile_base_link
- joint armbase1_support_joint: parent base_link -> mobile_base_link
- joint armbase2_support_joint: parent base_link -> mobile_base_link
- joint armbase3_support_joint: parent base_link -> mobile_base_link
- joint armbase4_support_joint: parent base_link -> mobile_base_link
- joint base_caster_left_joint: parent base_link -> mobile_base_link
- joint base_caster_right_joint: parent base_link -> mobile_base_link
- joint base_joint: child base_link -> mobile_base_link; parent base_footprint_link -> base_link
- joint base_left_wheel_joint: axis 0 1 0 -> (none); parent base_link -> mobile_base_link; type continuous -> fixed
- joint base_right_wheel_joint: axis 0 1 0 -> (none); parent base_link -> mobile_base_link; type continuous -> fixed
- joint realsense_joint: parent base_link -> mobile_base_link

Commit message: modified:   src/mapping/mapping/grid_publisher.py 	modified:   src/motion_control/motion_control/motion_control.py 	modified:   src/robp_interfaces/CMakeLists.txt 	new file:   src/robp_interfaces/msgs/Object.msg 	new file:   src/robp_interfaces/msgs/ObjectList.msg

File: src/snow_description/urdf/snow.urdf (robot description, URDF)
Before this commit: robot snow, 26 links, 25 joints
Links:
- removed link camera_link
- added link arm_camera_link; visual mesh filename=package://snow_description/meshes/camera_link.STL
Joints:
- joint camera_joint: child camera_link -> arm_camera_link
